Commit message: configured twist_mux pkg

File: install/robot_car_v2_description/share/robot_car_v2_description/urdf/robot_car_v2_urdf.urdf.xacro (robot description, xacro)
@@ -29,9 +29,4 @@
     </collision>
   </link>
-  <joint name="base_joint" type="fixed">
-    <parent link="base_footprint"/>
-    <child link="base_link" />
-    <origin xyz="0 0 0.033" rpy="0 0 0"/>
-  </joint>
   <link name="wheel_right_link">
     <inertial>
@@ -55,12 +50,5 @@
     </collision>
   </link>
-  <joint name="wheel_right_joint" type="continuous">
-    <origin xyz="0 -0.0701101849418637 0" rpy="0 0 0" />
-    <parent link="base_link" />
-    <child link="wheel_right_link" />
-    <axis xyz="0 1 0" />
-  </joint>
-  <link
-    name="wheel_left_link">
+  <link name="wheel_left_link">
     <inertial>
       <origin xyz="0 0.014 0" rpy="0 0 0" />
@@ -170,4 +158,15 @@
     </collision>
   </link>
+  <joint name="base_joint" type="fixed">
+    <parent link="base_footprint"/>
+    <child link="base_link" />
+    <origin xyz="0 0 0.033" rpy="0 0 0"/>
+  </joint>
+  <joint name="wheel_right_joint" type="continuous">
+    <origin xyz="0 -0.0701101849418637 0" rpy="0 0 0" />
+    <parent link="base_link" />
+    <child link="wheel_right_link" />
+    <axis xyz="0 1 0" />
+  </joint>
   <joint name="wheel_left_joint" type="continuous">
     <origin xyz="0 0.0701101849418642 0" rpy="0 0 0" />
@@ -200,6 +199,6 @@
     <axis xyz="0 0 0" />
   </joint>
-   <gazebo reference="base_link">
-        <material>Gazebo/Blue</material>
-    </gazebo>
+  <gazebo reference="base_link">
+    <material>Gazebo/Blue</material>
+  </gazebo>
 </robot>
